Commit message: Temp fix of robot joint's mass

File: ros2_grasp_service_demo/open_manipulator/open_manipulator_description/urdf/open_manipulator.xacro (robot description, xacro)
@@ -59,5 +59,5 @@
     <inertial>
       <origin xyz="1.0308393e-02 3.7743363e-04 1.0170197e-01" />
-      <mass value="1.3850917e-01" />
+      <mass value="1.3850917e-02" />
       <inertia ixx="3.3055381e-04" ixy="-9.7940978e-08" ixz="-3.8505711e-05"
                iyy="3.4290447e-04" iyz="-1.5717516e-06"
@@ -77,5 +77,5 @@
     <inertial>
       <origin xyz="9.0909590e-02 3.8929816e-04 2.2413279e-04" />
-      <mass value="1.3274562e-01" />
+      <mass value="1.3274562e-02" />
       <inertia ixx="3.0654178e-05" ixy="-1.2764155e-06" ixz="-2.6874417e-07"
                iyy="2.4230292e-04" iyz="1.1559550e-08"
@@ -95,5 +95,5 @@
     <inertial>
       <origin xyz="4.4206755e-02 3.6839985e-07 8.9142216e-03" />
-      <mass value="1.4327573e-01" />
+      <mass value="1.4327573e-02" />
       <inertia ixx="8.0870749e-05" ixy="0.0" ixz="-1.0157896e-06"
                iyy="7.5980465e-05" iyz="0.0"

Commit message: Fix gz physics

File: ros2_grasp_service_demo/open_manipulator/open_manipulator_description/urdf/open_manipulator.xacro (robot description, xacro)
@@ -59,5 +59,5 @@
     <inertial>
       <origin xyz="1.0308393e-02 3.7743363e-04 1.0170197e-01" />
-      <mass value="1.3850917e-02" />
+      <mass value="1.3850917e-01" />
       <inertia ixx="3.3055381e-04" ixy="-9.7940978e-08" ixz="-3.8505711e-05"
                iyy="3.4290447e-04" iyz="-1.5717516e-06"
@@ -77,5 +77,5 @@
     <inertial>
       <origin xyz="9.0909590e-02 3.8929816e-04 2.2413279e-04" />
-      <mass value="1.3274562e-02" />
+      <mass value="1.3274562e-01" />
       <inertia ixx="3.0654178e-05" ixy="-1.2764155e-06" ixz="-2.6874417e-07"
                iyy="2.4230292e-04" iyz="1.1559550e-08"
@@ -95,5 +95,5 @@
     <inertial>
       <origin xyz="4.4206755e-02 3.6839985e-07 8.9142216e-03" />
-      <mass value="1.4327573e-02" />
+      <mass value="1.4327573e-01" />
       <inertia ixx="8.0870749e-05" ixy="0.0" ixz="-1.0157896e-06"
                iyy="7.5980465e-05" iyz="0.0"
